File: LSwarm Firefly/LSwarm Firefly.kicad_pcb (KiCad board)
At the start: 2 copper layers, 50 x 50 mm, 83 parts, among them J2 Conn_01x06_Pin, J3 JST / BT2.0 Connector, J4 Conn_01x02_Pin, J5 Conn_01x06_Pin, Q1 AO3400A, Q7 AO3407A, SW1 MSK12C02, SW3 SKRPACE010, U1 LSM6DSRTR, U12 AP2112K-3.3, U2 STM32G473RCT6, U3 TPS61023DRLR, U4 SN74LVC1T45DBVR, U5 BMP581, U6 ESP32-C3-MINI-1U-N4

Commit message: sync
Parts:
- removed J2: Conn_01x06_Pin, Connector_PinHeader_2.54mm:PinHeader_1x06_P2.54mm_Vertical
- added D2: SS14, Diode_SMD:D_SMA, F.Cu at (39.8, 36.0)
- added J6: Conn_01x03_Pin, Connector_PinHeader_2.54mm:PinHeader_1x03_P2.54mm_Vertical, F.Cu at (6.25, 35.5)
- added J7: Conn_01x03_Pin, Connector_PinHeader_2.54mm:PinHeader_1x03_P2.54mm_Vertical, F.Cu at (2.25, 35.3)
- added J8: Conn_01x03_Pin, Connector_PinHeader_2.54mm:PinHeader_1x03_P2.54mm_Vertical, F.Cu at (44.0, 30.0)
- added J9: Conn_01x03_Pin, Connector_PinHeader_2.54mm:PinHeader_1x03_P2.54mm_Vertical, F.Cu at (48.0, 28.0)
- added Q2: AO3400A, Package_TO_SOT_SMD:SOT-23, F.Cu at (39.8, 41.8)
- added R13: 100, Resistor_SMD:R_0603_1608Metric, F.Cu at (36.3, 39.8)
- added R16: 4.7k, Resistor_SMD:R_0603_1608Metric, F.Cu at (36.2, 41.5)
- J3, LED1, LED2, LED3, LED4: moved to B.Cu
- J5: value Conn_01x06_Pin -> Conn_01x02_Pin; footprint Connector_PinHeader_2.54mm:PinHeader_1x06_P2.54mm_Vertical -> Connector_PinHeader_2.54mm:PinHeader_1x02_P2.54mm_Vertical
- moved J3 99.7 mm to (1.80, 18.2), turned to -90 degrees
- moved C1 97.2 mm to (8.00, 22.8)
- moved U3 90.8 mm to (13.2, 12.5), turned to 180 degrees
- moved L5 90.2 mm to (13.8, 9.00), turned to -90 degrees
- moved U12 83.7 mm to (11.6, 19.7)
- moved SW3 81.0 mm to (32.2, 2.00)
- moved C45 77.5 mm to (6.77, 6.77), turned to -135 degrees
- moved C71Ceramic1 77.1 mm to (4.00, 22.8)
- moved J4 74.5 mm to (28.0, 34.5)
- moved BUZZER2 73.3 mm to (35.0, 46.8)
- moved U4 72.3 mm to (12.7, 25.7), turned to 180 degrees
- moved D1 71.6 mm to (31.8, 36.3), turned to -90 degrees
- moved R32 70.6 mm to (24.8, 49.0), turned to 180 degrees
- moved R28 69.9 mm to (5.50, 16.8), turned to 180 degrees
- moved STATUS1 69.7 mm to (22.0, 5.50), turned to 90 degrees
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Connections:
- net RP2350_PB6_5.5V renamed STM32_PC4_5.5V
- J5 pad 1: STM32_SWCLK -> BATT_SW+
- J5 pad 2: STM32_SWDIO -> Net-(D2-A)
- R12 pad 1: STM32_PB4 -> STM32_PC2
- R27 pad 1: STM32_PB5 -> STM32_PC5
- U2 pad 10: unconnected-(U2-PC2-Pad10) -> STM32_PC2
- U2 pad 22: unconnected-(U2-PC4-Pad22) -> STM32_PC4
- U2 pad 23: unconnected-(U2-PC5-Pad23) -> STM32_PC5
- U2 pad 41: STM32_PC9 -> unconnected-(U2-PC9-Pad41)
- U2 pad 42: STM32_PA8 -> unconnected-(U2-PA8-Pad42)
- U2 pad 44: STM32_PA10 -> unconnected-(U2-PA10-Pad44)
- U2 pad 57: STM32_PB4 -> unconnected-(U2-PB4-Pad57)
- U2 pad 58: STM32_PB5 -> unconnected-(U2-PB5-Pad58)
- U2 pad 59: STM32_PB6 -> unconnected-(U2-PB6-Pad59)
- U4 pad 3: STM32_PB6 -> STM32_PC4
Routing:
- net +5V: track 0.00 -> 140.0 mm, vias 0 -> 7
- net GND: track 0.00 -> 111.1 mm, vias 0 -> 93
- net BATT_SW+: track 0.00 -> 65.0 mm
- net STM32_PA0: track 0.00 -> 57.0 mm, vias 0 -> 3
- net +3.3V: track 0.00 -> 43.3 mm, vias 0 -> 31
- net Net-(LED1-DOUT): track 0.00 -> 39.8 mm
- net Net-(LED2-DOUT): track 0.00 -> 39.3 mm, vias 0 -> 2
- net Net-(LED3-DOUT): track 0.00 -> 38.3 mm
- net STM32_TRACESWO: track 0.00 -> 37.3 mm, vias 0 -> 2
- net STM32_NRST: track 0.00 -> 31.5 mm, vias 0 -> 1
- net STM32_PA1: track 0.00 -> 31.3 mm, vias 0 -> 2
- net STM32_SWCLK: track 0.00 -> 31.2 mm, vias 0 -> 1
- net STM32_PA3: track 0.00 -> 30.6 mm, vias 0 -> 2
- net STM32_SWDIO: track 0.00 -> 29.8 mm, vias 0 -> 1
- net STM32_PC3: track 0.00 -> 29.2 mm, vias 0 -> 4
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- added copper zone on In2.Cu, net +3.3V
- added copper zone on In1.Cu, net GND
Other:
- outline, holes or cut-outs redrawn
- copper layers 2 -> 4
- board text added: "ESP32"
- board text added: "STM32"

Commit message: sync
Parts:
- moved R32 18.7 mm to (6.50, 45.2), turned to -45 degrees
- moved C64 8.81 mm to (19.5, 6.50), turned to 90 degrees
- moved R42 2.91 mm to (40.5, 25.2), turned to -90 degrees
- moved C57 1.60 mm to (38.8, 25.2), turned to 90 degrees
- moved C62 1.60 mm to (18.0, 6.47)
- moved C52 1.52 mm to (28.0, 44.5)
- moved R18 1.52 mm to (28.0, 46.2)
- moved C63 1.25 mm to (19.0, 9.75)
Routing:
- net Net-(LED2-DOUT): track 39.3 -> 43.8 mm
- net Net-(U6-IO2): track 8.79 -> 12.0 mm
- net STM32_PA0: track 57.0 -> 58.5 mm, vias 3 -> 5
- net STM32_PB8_BOOT: track 23.9 -> 24.8 mm
- net STM32_TRACESWO: track 37.3 -> 37.8 mm, vias 2 -> 1
Other:
- outline, holes or cut-outs redrawn

Commit message: sync
Parts:
- removed D2: SS14, Diode_SMD:D_SMA
- removed J5: Conn_01x02_Pin, Connector_PinHeader_2.54mm:PinHeader_1x02_P2.54mm_Vertical
- removed J6, J7, J8, J9: Conn_01x03_Pin, Connector_PinHeader_2.54mm:PinHeader_1x03_P2.54mm_Vertical
- removed Q2: AO3400A, Package_TO_SOT_SMD:SOT-23
- removed R13: 100, Resistor_SMD:R_0603_1608Metric
- removed R16: 4.7k, Resistor_SMD:R_0603_1608Metric
- added C49: 100uF, Capacitor_SMD:C_0603_1608Metric, F.Cu at (95.2, 60.5)
- added TP22: USB_DN, TestPoint:TestPoint_Pad_1.0x1.0mm, F.Cu at (41.1, 28.9)
- added TP23: USB_DP, TestPoint:TestPoint_Pad_1.0x1.0mm, F.Cu at (41.1, 32.0)
- added TP24: USB_DN, TestPoint:TestPoint_Pad_1.0x1.0mm, F.Cu at (41.1, 35.0)
- added TP25: USB_DP, TestPoint:TestPoint_Pad_1.0x1.0mm, F.Cu at (41.1, 38.1)
- added TP26: STM32_SWCLK, TestPoint:TestPoint_Pad_1.0x1.0mm, F.Cu at (5.25, 1.25)
- added TP27: STM32_SWDIO, TestPoint:TestPoint_Pad_1.0x1.0mm, F.Cu at (7.25, 1.25)
- added TP28: STM32_TRACESWO, TestPoint:TestPoint_Pad_1.0x1.0mm, F.Cu at (3.25, 1.25)
- added TP29: STM32_NRST, TestPoint:TestPoint_Pad_1.0x1.0mm, F.Cu at (2.50, 16.8)
- added TP30: Motor1, TestPoint:TestPoint_Pad_1.0x1.0mm, F.Cu at (44.2, 28.9)
- added TP31: Motor1, TestPoint:TestPoint_Pad_1.0x1.0mm, F.Cu at (44.2, 32.0)
- added TP32: Servo1, TestPoint:TestPoint_Pad_1.0x1.0mm, F.Cu at (44.2, 35.0)
- added TP33: Servo1, TestPoint:TestPoint_Pad_1.0x1.0mm, F.Cu at (44.2, 38.1)
- added TP34: ESP32_EN, TestPoint:TestPoint_Pad_1.0x1.0mm, F.Cu at (44.2, 41.1)
- added TP35: ESP32_EN, TestPoint:TestPoint_Pad_1.0x1.0mm, F.Cu at (47.2, 19.8)
- added TP36: ESP32_BOOT, TestPoint:TestPoint_Pad_1.0x1.0mm, F.Cu at (47.2, 22.8)
- added TP37: ESP32_BOOT, TestPoint:TestPoint_Pad_1.0x1.0mm, F.Cu at (47.2, 25.9)
- added TP38: ESP32_RX, TestPoint:TestPoint_Pad_1.0x1.0mm, F.Cu at (47.2, 28.9)
- added TP39: ESP32_RX, TestPoint:TestPoint_Pad_1.0x1.0mm, F.Cu at (47.2, 32.0)
- added TP40: ESP32_TX, TestPoint:TestPoint_Pad_1.0x1.0mm, F.Cu at (47.2, 35.0)
- added TP42: STM32_GND, TestPoint:TestPoint_Pad_1.0x1.0mm, F.Cu at (1.25, 4.00)
- added TP43: ESP32_TX, TestPoint:TestPoint_Pad_1.0x1.0mm, F.Cu at (50.3, 19.8)
- added TP44: LED_ARRAY, TestPoint:TestPoint_Pad_1.0x1.0mm, F.Cu at (50.3, 22.8)
- added TP45: LED_ARRAY, TestPoint:TestPoint_Pad_1.0x1.0mm, F.Cu at (7.50, 24.0)
- added TP46: BUZZ, TestPoint:TestPoint_Pad_1.0x1.0mm, F.Cu at (50.3, 28.9)
- added TP47: BUZZ, TestPoint:TestPoint_Pad_1.0x1.0mm, F.Cu at (9.50, 24.0)
- added TP48: VMON, TestPoint:TestPoint_Pad_1.0x1.0mm, F.Cu at (50.3, 35.0)
- added TP50: ServoPWM, TestPoint:TestPoint_Pad_1.0x1.0mm, F.Cu at (16.8, 52.0)
- added TP51: 5V, TestPoint:TestPoint_Pad_1.0x1.0mm, F.Cu at (50.3, 41.1)
- added TP52: 5V SIG, TestPoint:TestPoint_Pad_1.0x1.0mm, F.Cu at (53.3, 19.8)
- added TP53: 5V SIG, TestPoint:TestPoint_Pad_1.0x1.0mm, F.Cu at (53.3, 22.8)
- added TP54: DOUT1, TestPoint:TestPoint_Pad_1.0x1.0mm, F.Cu at (53.3, 25.9)
- added TP55: DIN1, TestPoint:TestPoint_Pad_1.0x1.0mm, F.Cu at (53.3, 28.9)
- added TP56: GND, TestPoint:TestPoint_Pad_1.0x1.0mm, F.Cu at (53.3, 32.0)
- added TP57: 5V, TestPoint:TestPoint_Pad_1.0x1.0mm, F.Cu at (53.3, 35.0)
- added TP58: 5V OUTPUT, TestPoint:TestPoint_Pad_2.0x2.0mm, F.Cu at (59.9, 20.3)
- added TP59: GND OUTPUT, TestPoint:TestPoint_Pad_2.0x2.0mm, F.Cu at (59.9, 24.3)
- added TP60: 5V, TestPoint:TestPoint_Pad_1.0x1.0mm, F.Cu at (53.3, 38.1)
- added TP61: DOUT2, TestPoint:TestPoint_Pad_1.0x1.0mm, F.Cu at (53.3, 41.1)
- added TP62: GND, TestPoint:TestPoint_Pad_1.0x1.0mm, F.Cu at (56.4, 19.8)
- added TP63: DOUT3, TestPoint:TestPoint_Pad_1.0x1.0mm, F.Cu at (56.4, 22.8)
- added TP64: 5V, TestPoint:TestPoint_Pad_1.0x1.0mm, F.Cu at (56.4, 25.9)
- added TP65: DIN2, TestPoint:TestPoint_Pad_1.0x1.0mm, F.Cu at (56.4, 28.9)
- added TP66: GND, TestPoint:TestPoint_Pad_1.0x1.0mm, F.Cu at (56.4, 32.0)
- added TP67: 5V, TestPoint:TestPoint_Pad_1.0x1.0mm, F.Cu at (56.4, 35.0)
- added TP68: DIN3, TestPoint:TestPoint_Pad_1.0x1.0mm, F.Cu at (56.4, 38.1)
- added TP69: GND, TestPoint:TestPoint_Pad_1.0x1.0mm, F.Cu at (56.4, 41.1)
- added TP70: 3.3V OUTPUT, TestPoint:TestPoint_Pad_2.0x2.0mm, F.Cu at (1.75, 51.8)
- added TP71: 3.3V INPUT, TestPoint:TestPoint_Pad_1.0x1.0mm, F.Cu at (1.25, 1.25)
- added TP72: 3.3V INPUT, TestPoint:TestPoint_Pad_2.0x2.0mm, F.Cu at (2.00, 27.0)
- added TP73: ServoVCC, TestPoint:TestPoint_Pad_1.0x1.0mm, F.Cu at (19.8, 52.0)
- added TP74: ServoGND, TestPoint:TestPoint_Pad_1.0x1.0mm, F.Cu at (22.8, 52.0)
- added TPe: VMON, TestPoint:TestPoint_Pad_1.0x1.0mm, F.Cu at (11.5, 24.0)
- J3, LED1, LED2, LED3, LED4: moved to F.Cu
- moved C45 115.2 mm to (103.5, 69.3), turned to 0 degrees
- moved C71Ceramic1 112.5 mm to (103.5, 75.3)
- moved R28 109.7 mm to (107.2, 58.0), turned to 0 degrees
- moved R36 106.7 mm to (111.2, 45.5), turned to 0 degrees
- moved R37 105.7 mm to (111.2, 48.0), turned to 0 degrees
- moved C63 105.1 mm to (103.5, 72.3), turned to 0 degrees
- moved R32 104.8 mm to (111.2, 40.4), turned to 0 degrees
- moved R17 102.4 mm to (107.2, 43.0), turned to 0 degrees
- moved C42 102.0 mm to (103.5, 63.3)
- moved C43 101.0 mm to (103.5, 66.3), turned to 0 degrees
- moved C65 97.0 mm to (103.2, 40.4), turned to 0 degrees
- moved C44 96.7 mm to (95.2, 50.5), turned to 0 degrees
- moved R9 95.2 mm to (103.2, 55.5)
- moved R19 94.0 mm to (107.2, 48.0)
- moved R10 93.9 mm to (103.2, 58.0)
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Connections:
- net STM32_NRST renamed Net-(U2-PG10-NRST)
- net STM32_PA9 renamed STM32_USB_VBUS
- net STM32_PB11 renamed BARO_INT
- net STM32_PB12 renamed BARO_CSB
- net STM32_PB13 renamed SENSOR_SCL
- net STM32_PB14 renamed SENSOR_SDO
- net STM32_PB15 renamed SENSOR_SDA
- net STM32_PC6 renamed IMU_INT2
- net STM32_PC7 renamed IMU_INT1
- net STM32_PC8 renamed IMU_CS
- C44 pad 2: +5V -> Net-(C44-Pad2)
- C46 pad 1: GND -> Net-(LED1-GND)
- C46 pad 2: +5V -> Net-(LED1-VDD)
- C47 pad 1: GND -> Net-(LED2-GND)
- C47 pad 2: +5V -> Net-(LED2-VDD)
- C48 pad 1: GND -> Net-(LED3-GND)
- C48 pad 2: +5V -> Net-(LED3-VDD)
- C52 pad 2: STM32_PA0 -> Net-(U6-EN)
- C71 pad 2: STM32_PB0 -> Net-(C71-Pad2)
- D6 pad 4: STM32_USB_DP -> Net-(D6-I/O2-Pad4)
- D6 pad 6: STM32_USB_DN -> Net-(D6-I/O1-Pad6)
- LED1 pad 1: GND -> Net-(LED1-GND)
- LED1 pad 3: +5V -> Net-(LED1-VDD)
- LED2 pad 1: GND -> Net-(LED2-GND)
- LED2 pad 2: Net-(LED1-DOUT) -> Net-(LED2-DIN)
- LED2 pad 3: +5V -> Net-(LED2-VDD)
- LED3 pad 1: GND -> Net-(LED3-GND)
- LED3 pad 2: Net-(LED2-DOUT) -> Net-(LED3-DIN)
- LED3 pad 3: +5V -> Net-(LED3-VDD)
- LED4 pad 1: GND -> Net-(LED4-GND)
- LED4 pad 2: Net-(LED3-DOUT) -> Net-(LED4-DIN)
- LED4 pad 3: +5V -> Net-(LED4-VDD)
- R12 pad 1: STM32_PC2 -> Net-(R12-Pad1)
- R18 pad 1: STM32_PA0 -> Net-(U6-EN)
- R19 pad 2: Net-(U4-B) -> Net-(U4-A)
- R25 pad 2: STM32_PB0 -> Net-(C71-Pad2)
- R26 pad 2: STM32_PB0 -> Net-(C71-Pad2)
- R27 pad 1: STM32_PC5 -> Net-(R27-Pad1)
- R9 pad 1: Net-(LED1-DIN) -> Net-(R9-Pad1)
- U2 pad 10: STM32_PC2 -> Net-(U2-PC2)
- U2 pad 11: STM32_PC3 -> Net-(U2-PC3)
- U2 pad 12: STM32_PA0 -> Net-(U2-PA0)
- U2 pad 13: STM32_PA1 -> Net-(U2-PA1)
- U2 pad 14: STM32_PA2 -> Net-(U2-PA2)
- U2 pad 17: STM32_PA3 -> Net-(U2-PA3)
- U2 pad 22: STM32_PC4 -> Net-(U2-PC4)
- U2 pad 23: STM32_PC5 -> Net-(U2-PC5)
- U2 pad 24: STM32_PB0 -> Net-(U2-PB0)
- U2 pad 45: STM32_USB_DN -> Net-(U2-PA11)
- U2 pad 46: STM32_USB_DP -> Net-(U2-PA12)
- U2 pad 49: STM32_SWDIO -> Net-(U2-PA13)
- U2 pad 50: STM32_SWCLK -> Net-(U2-PA14)
- U2 pad 56: STM32_TRACESWO -> Net-(U2-PB3)
- U4 pad 1: +3.3V -> +5V
- U4 pad 2: GND -> +3.3V
- U4 pad 3: STM32_PC4 -> Net-(U4-A)
- U4 pad 5: +3.3V -> GND
- U4 pad 6: +5V -> +3.3V
- U6 pad 23: STM32_PA1 -> Net-(U6-IO9)
- U6 pad 30: STM32_PA2 -> Net-(U6-RXD0)
- U6 pad 31: STM32_PA3 -> Net-(U6-TXD0)
- U6 pad 8: STM32_PA0 -> Net-(U6-EN)
Routing:
- net +5V: track 140.0 -> 0.00 mm, vias 7 -> 0
- net GND: track 111.3 -> 0.00 mm, vias 93 -> 0
- net BATT_SW+: track 65.0 -> 0.00 mm
- net STM32_PA0: track 58.5 -> 0.00 mm, vias 5 -> 0
- net Net-(LED2-DOUT): track 43.8 -> 0.00 mm, vias 2 -> 0
- net +3.3V: track 42.9 -> 0.00 mm, vias 31 -> 0
- net Net-(LED1-DOUT): track 40.1 -> 0.00 mm
- net Net-(LED3-DOUT): track 38.4 -> 0.00 mm
- net STM32_TRACESWO: track 37.8 -> 0.00 mm, vias 1 -> 0
- net STM32_PA1: track 31.3 -> 0.00 mm, vias 2 -> 0
- net STM32_SWCLK: track 31.2 -> 0.00 mm, vias 1 -> 0
- net STM32_PA3: track 30.6 -> 0.00 mm, vias 2 -> 0
- net STM32_SWDIO: track 29.8 -> 0.00 mm, vias 1 -> 0
- net STM32_PC3: track 29.2 -> 0.00 mm, vias 4 -> 0
- net STM32_PC4: track 28.7 -> 0.00 mm, vias 2 -> 0
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- removed copper zone on In2.Cu, net +3.3V
- removed copper zone on In1.Cu, net GND
Other:
- board size 50 x 50 mm -> 25 x 75 mm
- board text added: "3.3V"
- board text added: "BUZZ"
- board text added: "CLK"
- board text added: "DIO"
- board text added: "GND"
- board text added: "LED"
- board text added: "NRST"
- board text added: "SWO"
- board text added: "VMON"
- board text removed: "ESP32"
- board text removed: "STM32"
