File: LSwarm Firefly/LSwarm Firefly.kicad_pcb (KiCad board)
At the start: 4 copper layers, 25 x 75 mm, 134 parts, among them J3 JST / BT2.0 Connector, J4 Conn_01x02_Pin, Q1 AO3400A, Q7 AO3407A, SW1 MSK12C02, SW3 SKRPACE010, U1 LSM6DSRTR, U12 AP2112K-3.3, U2 STM32G473RCT6, U3 TPS61023DRLR, U4 SN74LVC1T45DBVR, U5 BMP581, U6 ESP32-C3-MINI-1U-N4

Commit message: sync
Parts:
- removed D1: SS14, Diode_SMD:D_SMA
- removed J4: Conn_01x02_Pin, Connector_PinHeader_2.54mm:PinHeader_1x02_P2.54mm_Vertical
- removed Q1: AO3400A, Package_TO_SOT_SMD:SOT-23
- removed R11: 4.7k, Resistor_SMD:R_0603_1608Metric
- removed R12: 100, Resistor_SMD:R_0603_1608Metric
- removed TP22, TP24: USB_DN, TestPoint:TestPoint_Pad_1.0x1.0mm
- removed TP23, TP25: USB_DP, TestPoint:TestPoint_Pad_1.0x1.0mm
- removed TP30, TP31: Motor1, TestPoint:TestPoint_Pad_1.0x1.0mm
- added C61: 100nF, Capacitor_SMD:C_0603_1608Metric, F.Cu at (10.9, 97.2)
- added C69: 100nF, Capacitor_SMD:C_0603_1608Metric, F.Cu at (13.5, 97.2)
- added C70: 100nF, Capacitor_SMD:C_0603_1608Metric, F.Cu at (16.0, 97.2)
- added C72: 10uF, Capacitor_SMD:C_0603_1608Metric, F.Cu at (18.5, 97.2)
- added C73: 1uF, Capacitor_SMD:C_0603_1608Metric, F.Cu at (21.0, 97.2)
- added R34: 10k, Resistor_SMD:R_0603_1608Metric, F.Cu at (23.5, 97.2)
- added R35: 47k, Resistor_SMD:R_0603_1608Metric, F.Cu at (26.0, 97.2)
- added R39: 47k, Resistor_SMD:R_0603_1608Metric, F.Cu at (28.5, 97.2)
- added R43: 10k, Resistor_SMD:R_0603_1608Metric, F.Cu at (31.0, 97.2)
- added TP100: M_INHB, TestPoint:TestPoint_Pad_1.0x1.0mm, F.Cu at (-1.50, 91.8)
- added TP101: M_INHA, TestPoint:TestPoint_Pad_1.0x1.0mm, F.Cu at (-1.50, 93.8)
- added TP102: M_nFAULT, TestPoint:TestPoint_Pad_1.0x1.0mm, F.Cu at (45.4, 36.0)
- added TP103: M_nFAULT, TestPoint:TestPoint_Pad_1.0x1.0mm, F.Cu at (45.4, 39.0)
- added TP104: M_SOB, TestPoint:TestPoint_Pad_1.0x1.0mm, F.Cu at (-4.00, 18.2)
- added TP41: M_INLC, TestPoint:TestPoint_Pad_1.0x1.0mm, F.Cu at (42.8, 45.8)
- added TP75: STATUS, TestPoint:TestPoint_Pad_1.0x1.0mm, F.Cu at (13.2, 4.50)
- added TP76: STATUS, TestPoint:TestPoint_Pad_1.0x1.0mm, F.Cu at (10.2, 35.3)
- added TP79: GND INPUT, TestPoint:TestPoint_Pad_1.0x1.0mm, F.Cu at (25.5, 35.3)
- added TP80: GND INPUT, TestPoint:TestPoint_Pad_1.0x1.0mm, F.Cu at (25.5, 4.50)
- added TP81: GND INPUT, TestPoint:TestPoint_Pad_1.0x1.0mm, F.Cu at (25.5, 66.0)
- added TP83: M_SOA, TestPoint:TestPoint_Pad_1.0x1.0mm, F.Cu at (-4.00, 16.2)
- added TP84: M_SOC, TestPoint:TestPoint_Pad_1.0x1.0mm, F.Cu at (33.2, 91.0)
- added TP85: M_SOB, TestPoint:TestPoint_Pad_1.0x1.0mm, F.Cu at (33.2, 89.0)
- added TP86: M_SOA, TestPoint:TestPoint_Pad_1.0x1.0mm, F.Cu at (33.2, 87.0)
- added TP87: MotorA, TestPoint:TestPoint_Pad_1.0x1.0mm, F.Cu at (2.00, 86.8)
- added TP88: MotorB, TestPoint:TestPoint_Pad_1.0x1.0mm, F.Cu at (2.00, 84.8)
- added TP89: MotorC, TestPoint:TestPoint_Pad_1.0x1.0mm, F.Cu at (2.00, 82.8)
- added TP90: M_INLA, TestPoint:TestPoint_Pad_1.0x1.0mm, F.Cu at (34.2, 10.0)
- added TP91: M_nSleep, TestPoint:TestPoint_Pad_1.0x1.0mm, F.Cu at (39.2, 32.9)
- added TP92: M_nSleep, TestPoint:TestPoint_Pad_1.0x1.0mm, F.Cu at (39.2, 36.0)
- added TP93: M_INHC, TestPoint:TestPoint_Pad_1.0x1.0mm, F.Cu at (39.2, 39.0)
- added TP94: M_INHB, TestPoint:TestPoint_Pad_1.0x1.0mm, F.Cu at (39.2, 42.0)
- added TP95: M_INHA, TestPoint:TestPoint_Pad_1.0x1.0mm, F.Cu at (34.2, 13.1)
- added TP96: M_INLC, TestPoint:TestPoint_Pad_1.0x1.0mm, F.Cu at (2.00, 98.5)
- added TP97: M_INLB, TestPoint:TestPoint_Pad_1.0x1.0mm, F.Cu at (2.00, 96.5)
- added TP98: M_INLA, TestPoint:TestPoint_Pad_1.0x1.0mm, F.Cu at (2.00, 94.5)
- added TP99: M_INHC, TestPoint:TestPoint_Pad_1.0x1.0mm, F.Cu at (-1.50, 89.8)
- added U7: DRV8311HRRWR, easyeda2kicad:QFN-24_L3.0-W3.0-P0.40-TL-EP1.9_TI_RRW0024A, F.Cu at (14.8, 86.3)
- J3: moved to B.Cu
- TP42: value STM32_GND -> M_INLB
- TP57: value 5V -> M_SOC
- TP58, TP59, TP70, TP72: footprint TestPoint:TestPoint_Pad_2.0x2.0mm -> TestPoint:TestPoint_Pad_1.0x1.0mm
- moved R25 107.5 mm to (5.25, 84.8), turned to 180 degrees
- moved R26 107.2 mm to (5.25, 86.2), turned to 180 degrees
- moved C71 104.8 mm to (5.25, 87.8), turned to 180 degrees
- moved R36 103.7 mm to (13.0, 78.8), turned to -90 degrees
- moved C66 103.6 mm to (4.75, 75.2), turned to 90 degrees
- moved R37 102.6 mm to (14.2, 81.5), turned to 180 degrees
- moved R27 99.6 mm to (7.75, 50.0)
- moved C54 99.3 mm to (5.02, 13.7), turned to 90 degrees
- moved R19 99.3 mm to (10.8, 71.5), turned to -90 degrees
- moved C67 97.5 mm to (10.5, 75.7), turned to 90 degrees
- moved R9 95.5 mm to (8.32, 66.7)
- moved R41 95.5 mm to (19.8, 25.5), turned to 180 degrees
- moved R10 95.0 mm to (10.3, 37.8), turned to 180 degrees
- moved R38 95.0 mm to (22.2, 17.1), turned to 180 degrees
- moved R33 95.0 mm to (16.2, 43.8), turned to 180 degrees
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- renumbered TPe to TP49
Connections:
- C44 pad 2: Net-(C44-Pad2) -> +5V
- D6 pad 4: Net-(D6-I/O2-Pad4) -> USB_DP
- D6 pad 6: Net-(D6-I/O1-Pad6) -> USB_DN
- R10 pad 2: STM32_PB7 -> Net-(R10-Pad2)
- TP33 pad 1: Net-(U2-PC3) -> Net-(U2-PB4)
- TP42 pad 1: GND -> Net-(U2-PC11)
- TP57 pad 1: Net-(C44-Pad2) -> Net-(U2-PB1)
- U2 pad 10: Net-(U2-PC2) -> unconnected-(U2-PC2-Pad10)
- U2 pad 11: Net-(U2-PC3) -> unconnected-(U2-PC3-Pad11)
- U2 pad 18: unconnected-(U2-PA4-Pad18) -> Net-(U2-PA4)
- U2 pad 20: unconnected-(U2-PA6-Pad20) -> Net-(U2-PA6)
- U2 pad 21: unconnected-(U2-PA7-Pad21) -> Net-(U2-PA7)
- U2 pad 25: unconnected-(U2-PB1-Pad25) -> Net-(U2-PB1)
- U2 pad 38: IMU_INT2 -> Net-(U2-PC6)
- U2 pad 39: IMU_INT1 -> Net-(U2-PC7)
- U2 pad 40: IMU_CS -> Net-(U2-PC8)
- U2 pad 41: unconnected-(U2-PC9-Pad41) -> IMU_INT2
- U2 pad 42: unconnected-(U2-PA8-Pad42) -> IMU_INT1
- U2 pad 43: STM32_USB_VBUS -> IMU_CS
- U2 pad 44: unconnected-(U2-PA10-Pad44) -> STM32_USB_VBUS
- U2 pad 45: Net-(U2-PA11) -> USB_DN
- U2 pad 46: Net-(U2-PA12) -> USB_DP
- U2 pad 52: unconnected-(U2-PC10-Pad52) -> Net-(U2-PC10)
- U2 pad 53: unconnected-(U2-PC11-Pad53) -> Net-(U2-PC11)
- U2 pad 54: unconnected-(U2-PC12-Pad54) -> Net-(U2-PC12)
- U2 pad 57: unconnected-(U2-PB4-Pad57) -> Net-(U2-PB4)
- U2 pad 59: unconnected-(U2-PB6-Pad59) -> Net-(U2-PB6)
- U2 pad 60: STM32_PB7 -> Net-(U2-PB7)
Routing:
- net GND: track 0.00 -> 92.8 mm, vias 0 -> 83
- net BATT_SW+: track 0.00 -> 50.9 mm
- net +3.3V: track 0.00 -> 36.5 mm, vias 0 -> 33
- net Net-(U6-EN): track 0.00 -> 32.9 mm
- net Net-(TP32-Pad1): track 0.00 -> 25.5 mm, vias 0 -> 2
- net SENSOR_SDA: track 0.00 -> 22.1 mm, vias 0 -> 3
- net IMU_CS: track 0.00 -> 21.2 mm, vias 0 -> 2
- net SENSOR_SDO: track 0.00 -> 20.2 mm, vias 0 -> 3
- net Net-(C27-Pad2): track 0.00 -> 19.9 mm, vias 0 -> 1
- net +5V: track 0.00 -> 19.7 mm
- net IMU_INT1: track 0.00 -> 18.9 mm, vias 0 -> 2
- net USB_VBUS: track 0.00 -> 18.5 mm
- net SENSOR_SCL: track 0.00 -> 17.1 mm, vias 0 -> 3
- net Net-(U6-RXD0): track 0.00 -> 15.7 mm
- net Net-(U6-TXD0): track 0.00 -> 15.0 mm
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- added copper zone on In2.Cu, net +3.3V
- added copper zone on In1.Cu, net GND
Other:
- board size 25 x 75 mm -> 73.7 x 92 mm
- board text added: "BOOT"
- board text added: "EN"
- board text added: "LED ARRAY"
- board text added: "MOTOR"
- board text added: "Motor"
- board text added: "RX"
- board text added: "SERVO"
- board text added: "STAT"
- board text added: "STATUS"
- board text added: "TX"

Commit message: sync
Parts:
- removed C27: 10nF, Capacitor_SMD:C_0603_1608Metric
- removed D6: USBLC6-2SC6_C2687116, easyeda2kicad:SOT-23-6_L2.9-W1.6-P0.95-LS2.8-BL
- removed J3: JST / BT2.0 Connector, Connector_JST:JST_PH_S2B-PH-K_1x02_P2.00mm_Horizontal
- removed R14, R15: 100k, Resistor_SMD:R_0603_1608Metric
- removed R38, R41: 5.1k, Resistor_SMD:R_0603_1608Metric
- removed TP100, TP94: M_INHB, TestPoint:TestPoint_Pad_1.0x1.0mm
- removed TP101, TP95: M_INHA, TestPoint:TestPoint_Pad_1.0x1.0mm
- removed TP102, TP103: M_nFAULT, TestPoint:TestPoint_Pad_1.0x1.0mm
- removed TP104, TP85: M_SOB, TestPoint:TestPoint_Pad_1.0x1.0mm
- removed TP32, TP33: Servo1, TestPoint:TestPoint_Pad_1.0x1.0mm
- removed TP41, TP96: M_INLC, TestPoint:TestPoint_Pad_1.0x1.0mm
- removed TP42, TP97: M_INLB, TestPoint:TestPoint_Pad_1.0x1.0mm
- removed TP48, TP49: VMON, TestPoint:TestPoint_Pad_1.0x1.0mm
- removed TP57, TP84: M_SOC, TestPoint:TestPoint_Pad_1.0x1.0mm
- removed TP70: 3.3V OUTPUT, TestPoint:TestPoint_Pad_1.0x1.0mm
- removed TP81: GND INPUT, TestPoint:TestPoint_Pad_1.0x1.0mm
- removed TP83, TP86: M_SOA, TestPoint:TestPoint_Pad_1.0x1.0mm
- removed TP90, TP98: M_INLA, TestPoint:TestPoint_Pad_1.0x1.0mm
- removed TP91, TP92: M_nSleep, TestPoint:TestPoint_Pad_1.0x1.0mm
- removed TP93, TP99: M_INHC, TestPoint:TestPoint_Pad_1.0x1.0mm
- removed USB2: USB-TYPE-C-018, easyeda2kicad:USB-C_SMD-TYPE-C-31-M-12
- added G***: LOGO, LOGO, F.Cu at (20.7, 42.3)
- added J1: Conn_01x02_Socket, Connector_PinHeader_1.00mm:PinHeader_1x02_P1.00mm_Vertical, F.Cu at (5.52, 23.1)
- added J2: Conn_01x02_Socket, Connector_PinHeader_1.00mm:PinHeader_1x02_P1.00mm_Vertical, F.Cu at (4.56, 24.5)
- added U8: DW3110TR13, easyeda2kicad:WLCSP-53_L3.5-W3.0_DW3110TR13, F.Cu at (6.05, 45.8)
- C1, C42, C44, C45, C49, C61, C65, C66, C67, C69, C70, C71, C71Ceramic1, C72, C73, L5, Q7, R17, R19, R25, R26, R28, R34, R35, R36, R37, R39, R43, R9, SW1, TP34, TP36, TP38, TP40, TP44, TP50, TP52, TP58, TP59, TP72, TP73, TP74, TP76, TP79, TP87, TP88, TP89, U12, U3, U4, U7: moved to B.Cu
- moved R39 90.9 mm to (14.2, 7.38), turned to 180 degrees
- moved R35 89.1 mm to (14.2, 8.88), turned to 180 degrees
- moved R34 87.3 mm to (13.7, 10.4), turned to 180 degrees
- moved C69 85.3 mm to (8.18, 12.0), turned to 180 degrees
- moved R43 84.8 mm to (12.0, 14.5), turned to 180 degrees
- moved TP73 84.6 mm to (20.6, 4.50), turned to -90 degrees
- moved TP74 84.6 mm to (22.6, 4.50), turned to -90 degrees
- moved TP50 84.6 mm to (18.6, 4.50), turned to 0 degrees
- moved C61 84.2 mm to (11.5, 13.0), turned to 180 degrees
- moved C70 84.0 mm to (8.19, 13.5), turned to 0 degrees
- moved C73 83.7 mm to (14.2, 13.8)
- moved C72 81.5 mm to (11.7, 16.0), turned to 0 degrees
- moved C49 79.6 mm to (22.2, 6.50)
- moved R37 78.1 mm to (27.2, 4.50), turned to 0 degrees
- moved U7 77.6 mm to (10.3, 8.88), turned to 90 degrees
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Connections:
- C71 pad 2: Net-(C71-Pad2) -> V_MON
- C73 pad 2: Net-(U7-AVDD) -> M_nFAULT
- R25 pad 2: Net-(C71-Pad2) -> V_MON
- R26 pad 2: Net-(C71-Pad2) -> V_MON
- R34 pad 2: Net-(U7-nSLEEP) -> M_nSLEEP
- R43 pad 1: Net-(U7-AVDD) -> M_nFAULT
- TP50 pad 1: Net-(TP32-Pad1) -> SERVO_PWM
- U2 pad 18: Net-(U2-PA4) -> M_nSLEEP
- U2 pad 20: Net-(U2-PA6) -> M_SOA
- U2 pad 21: Net-(U2-PA7) -> M_SOB
- U2 pad 24: Net-(U2-PB0) -> V_MON
- U2 pad 25: Net-(U2-PB1) -> M_SOC
- U2 pad 38: Net-(U2-PC6) -> M_INHA
- U2 pad 39: Net-(U2-PC7) -> M_INHB
- U2 pad 40: Net-(U2-PC8) -> M_INHC
- U2 pad 45: USB_DN -> unconnected-(U2-PA11-Pad45)
- U2 pad 46: USB_DP -> unconnected-(U2-PA12-Pad46)
- U2 pad 52: Net-(U2-PC10) -> M_INLA
- U2 pad 53: Net-(U2-PC11) -> M_INLB
- U2 pad 54: Net-(U2-PC12) -> M_INLC
- U2 pad 57: Net-(U2-PB4) -> SERVO_PWM
- U2 pad 59: Net-(U2-PB6) -> M_nFAULT
- U7 pad 1: Net-(U7-AVDD) -> M_nFAULT
- U7 pad 13: Net-(U7-INHC) -> M_INHC
- U7 pad 14: Net-(U7-INHB) -> M_INHB
- U7 pad 15: Net-(U7-INHA) -> M_INHA
- U7 pad 17: Net-(U7-AVDD) -> M_nFAULT
- U7 pad 18: Net-(U7-INLA) -> M_INLA
- U7 pad 19: Net-(U7-INLB) -> M_INLB
- U7 pad 20: Net-(U7-INLC) -> M_INLC
- U7 pad 24: Net-(U7-nSLEEP) -> M_nSLEEP
- U7 pad 3: Net-(U7-SOC) -> M_SOC
- U7 pad 4: Net-(U7-SOB) -> M_SOB
- U7 pad 5: Net-(U7-SOA) -> M_SOA
Routing:
- net M_INHC: track 0.00 -> 31.9 mm, vias 0 -> 1
- net M_INHB: track 0.00 -> 31.8 mm, vias 0 -> 1
- net M_INHA: track 0.00 -> 31.4 mm, vias 0 -> 1
- net Net-(TP32-Pad1): track 25.5 -> 0.00 mm, vias 2 -> 0
- net M_nFAULT: track 0.00 -> 23.5 mm, vias 0 -> 1
- net GND: track 92.8 -> 113.1 mm, vias 83 -> 69
- net Net-(C27-Pad2): track 19.9 -> 0.00 mm, vias 1 -> 0
- net USB_VBUS: track 18.5 -> 0.00 mm
- net M_INLA: track 0.00 -> 13.6 mm, vias 0 -> 1
- net V_MON: track 0.00 -> 13.4 mm, vias 0 -> 1
- net STM32_USB_VBUS: track 13.4 -> 0.00 mm, vias 2 -> 0
- net M_INLB: track 0.00 -> 11.9 mm, vias 0 -> 1
- net +5V: track 19.7 -> 31.1 mm, vias 0 -> 1
- net M_nSLEEP: track 0.00 -> 10.9 mm, vias 0 -> 1
- net M_INLC: track 0.00 -> 10.6 mm, vias 0 -> 1
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Other:
- board size 73.7 x 92 mm -> 74.1 x 61.2 mm
- board text removed: "Motor"
- board text removed: "VMON"

Commit message: sync
Parts:
- removed U8: DW3110TR13, easyeda2kicad:WLCSP-53_L3.5-W3.0_DW3110TR13
- added C76: 10uF, Capacitor_SMD:C_0603_1608Metric, B.Cu at (8.98, 47.8)
- added C79: 100nf, Capacitor_SMD:C_0603_1608Metric, B.Cu at (8.95, 53.0)
- added C80: 100nf, Capacitor_SMD:C_0603_1608Metric, B.Cu at (8.97, 51.3)
- added C81: 100nf, Capacitor_SMD:C_0603_1608Metric, B.Cu at (8.97, 49.5)
- added L1: MPZ2012S601AT000, easyeda2kicad:L0805, B.Cu at (9.75, 44.0)
- added R41: 10k, Resistor_SMD:R_0603_1608Metric, B.Cu at (27.5, 47.3)
- added R44: 100k, Resistor_SMD:R_0603_1608Metric, B.Cu at (27.5, 55.8)
- added U11: BU03, easyeda2kicad:WIRELM-SMD_BU03, B.Cu at (18.8, 51.8)
- TP46: moved to B.Cu
- moved BUZZER2 18.8 mm to (25.5, 55.2)
- moved C55 18.2 mm to (9.07, 57.8), turned to 180 degrees
- moved R32 16.1 mm to (12.1, 57.8)
- moved R18 14.7 mm to (15.1, 57.8), turned to 180 degrees
- moved C52 14.0 mm to (18.1, 57.8), turned to 180 degrees
- moved R27 13.7 mm to (21.1, 53.0)
- moved TP46 8.49 mm to (6.50, 58.0), turned to 90 degrees
- moved U6 7.55 mm to (10.7, 50.0), turned to 90 degrees
- moved G*** 5.64 mm to (22.0, 47.8)
- moved R33 2.39 mm to (17.5, 45.8), turned to -90 degrees
Connections:
- U6 pad 13: unconnected-(U6-IO1-Pad13) -> DW_WAKEUP
- U6 pad 16: unconnected-(U6-IO10-Pad16) -> DW_RST
- U6 pad 18: unconnected-(U6-IO4-Pad18) -> DW_MISO
- U6 pad 19: unconnected-(U6-IO5-Pad19) -> DW_MOSI
- U6 pad 20: unconnected-(U6-IO6-Pad20) -> DW_CLK
- U6 pad 21: unconnected-(U6-IO7-Pad21) -> DW_Sn
- U6 pad 6: unconnected-(U6-IO3-Pad6) -> DW_IRQ
Routing:
- net GND: track 113.1 -> 166.5 mm
- net DW_IRQ: track 0.00 -> 18.9 mm, vias 0 -> 1
- net UW_3.3V: track 0.00 -> 18.8 mm
- net Net-(R27-Pad1): track 2.53 -> 18.1 mm, vias 0 -> 1
- net DW_Sn: track 0.00 -> 12.4 mm, vias 0 -> 1
- net DW_CLK: track 0.00 -> 11.5 mm, vias 0 -> 1
- net +3.3V: track 45.4 -> 56.3 mm
- net DW_MISO: track 0.00 -> 9.91 mm, vias 0 -> 1
- net DW_MOSI: track 0.00 -> 9.66 mm, vias 0 -> 1
- net Net-(U6-TXD0): track 14.9 -> 7.12 mm
- net Net-(U6-RXD0): track 15.9 -> 8.65 mm
- net DW_RST: track 0.00 -> 6.08 mm, vias 0 -> 1
- net Net-(U6-EN): track 32.8 -> 38.7 mm, vias 1 -> 3
- net DW_WAKEUP: track 0.00 -> 4.96 mm, vias 0 -> 1
- net Net-(U6-IO9): track 13.7 -> 17.9 mm
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
Commit message: sync
Parts:
- removed SW1: MSK12C02, easyeda2kicad:SW-TH_MSK12C02
- removed TP75: STATUS, TestPoint:TestPoint_Pad_1.0x1.0mm
- added C77: 100nF, Capacitor_SMD:C_0603_1608Metric, F.Cu at (10.2, 25.0)
- added C78: 1uF, Capacitor_SMD:C_0603_1608Metric, F.Cu at (8.00, 25.0)
- added C82: 100nF, Capacitor_SMD:C_0603_1608Metric, F.Cu at (21.1, 40.1)
- added C83: 1uF, Capacitor_SMD:C_0603_1608Metric, F.Cu at (21.1, 41.6)
- added R38: 4.7k, Resistor_SMD:R_0603_1608Metric, F.Cu at (12.8, 27.8)
- added R40: 4.7k, Resistor_SMD:R_0603_1608Metric, F.Cu at (13.3, 23.8)
- added R45: 4.7k, Resistor_SMD:R_0603_1608Metric, F.Cu at (16.8, 39.5)
- added R46: 4.7k, Resistor_SMD:R_0603_1608Metric, F.Cu at (16.8, 41.0)
- added SW2: MINI MSK12CO2, easyeda2kicad:SW-SMD_MSK12CO2, B.Cu at (7.97, 26.2)
- added TP77: STATUS, TestPoint:TestPoint_Pad_1.0x1.0mm, F.Cu at (13.0, 4.50)
- added U8: MMC5603NJ, easyeda2kicad:FLIPCHIP-4_L0.8-W0.8-R2-C2-P0.40-TL, F.Cu at (12.6, 25.8)
- added U9: MMC5603NJ, easyeda2kicad:FLIPCHIP-4_L0.8-W0.8-R2-C2-P0.40-TL, F.Cu at (18.8, 40.3)
- moved G*** 2.58 mm to (22.3, 45.2), turned to 180 degrees
- moved U11 0.42 mm to (18.8, 51.3)
- moved J1 0.30 mm to (5.45, 22.8)
- moved J2 0.30 mm to (4.49, 24.2)
Connections:
- C69 pad 2: BATT_SW+ -> BATT+
- C70 pad 1: BATT_SW+ -> BATT+
- U2 pad 51: unconnected-(U2-PA15-Pad51) -> STM_MAG_SCL
- U2 pad 58: unconnected-(U2-PB5-Pad58) -> Net-(U2-PB5)
- U2 pad 60: Net-(U2-PB7) -> STM_MAG_SDA
- U6 pad 26: unconnected-(U6-IO18-Pad26) -> ESP32_MAG_SDA
- U6 pad 27: unconnected-(U6-IO19-Pad27) -> ESP32_MAG_SCL
- U7 pad 7: BATT_SW+ -> BATT+
- U7 pad 8: BATT_SW+ -> BATT+
Routing:
- net STM_MAG_SDA: track 0.00 -> 42.3 mm, vias 0 -> 4
- net STM_MAG_SCL: track 0.00 -> 17.3 mm
- net +3.3V: track 56.3 -> 67.8 mm, vias 26 -> 30
- net BATT_SW+: track 49.3 -> 39.6 mm
- net ESP32_MAG_SDA: track 0.00 -> 8.75 mm, vias 0 -> 2
- net Net-(U2-PB5): track 0.00 -> 8.52 mm
- net Net-(U2-PB7): track 7.80 -> 0.00 mm
- net ESP32_MAG_SCL: track 0.00 -> 7.76 mm, vias 0 -> 2
- net BATT+: track 9.13 -> 16.6 mm
- net GND: track 166.5 -> 172.2 mm, vias 69 -> 71
- net Net-(C77-Pad2): track 0.00 -> 1.79 mm
- net Net-(C82-Pad2): track 0.00 -> 1.50 mm
- net STM32_PB8_BOOT: track 17.4 -> 18.2 mm
- net Net-(R17-Pad1): track 1.98 -> 2.78 mm
