File: LSwarm Firefly/LSwarm Firefly.kicad_sch (KiCad schematic)
At the start: 90 parts, among them J3 JST / BT2.0 Connector, J4 Conn_01x02_Pin, J5 Conn_01x02_Pin, J6 Conn_01x03_Pin, J7 Conn_01x03_Pin, J8 Conn_01x03_Pin, J9 Conn_01x03_Pin, Q1 AO3400A, Q2 AO3400A, Q7 AO3407A, SW1 MSK12C02, SW3 SKRPACE010, U1 LSM6DSRTR, U12 AP2112K-3.3, U2 STM32G473RCT6, U3 TPS61023DRLR, U4 SN74LVC1T45DBVR, U5 BMP581, U6 ESP32-C3-MINI-1U-N4

Commit message: sync
Connections:
- net STM32_PC3: now also R13.1
- net STM32_PC2: now reaches U2.10 (PC2)
- net STM32_PC2: now also R12.1
- net STM32_PC4: now reaches U2.22 (PC4)
- net STM32_PC4: now also U4.3 (A)
- net STM32_PC5: now reaches U2.23 (PC5)
- net STM32_PC5: now also R27.1
- net RP2350_PB6_5.5V renamed STM32_PC4_5.5V
- net STM32_PA10: no longer names the net of U2.44 (PA10)
- net STM32_PA8: no longer names the net of U2.42 (PA8)
- removed net STM32_PB4: R12.1, R13.1, U2.57 (PB4)
- net STM32_PB5: no longer names the net of U2.58 (PB5)
- net STM32_PB5: no longer R27.1
- net STM32_PB6: no longer names the net of U2.59 (PB6)
- net STM32_PB6: no longer U4.3 (A)
- net STM32_PC9: no longer names the net of U2.41 (PC9)
- no-connect marks 40 -> 41
Other:
- note added: "MOTOR 1"
- note added: "MOTOR 2"
- note removed: "MOTOR"

Commit message: sync
Parts:
- removed D2: SS14, Diode_SMD:D_SMA, symbol Diode:SS14
- removed J5: Conn_01x02_Pin, Connector_PinHeader_2.54mm:PinHeader_1x02_P2.54mm_Vertical, symbol Connector:Conn_01x02_Pin
- removed J6, J7, J8, J9: Conn_01x03_Pin, Connector_PinHeader_2.54mm:PinHeader_1x03_P2.54mm_Vertical, symbol Connector:Conn_01x03_Pin
- removed Q2: AO3400A, Package_TO_SOT_SMD:SOT-23, symbol Transistor_FET:AO3400A
- removed R13: 100, Resistor_SMD:R_0603_1608Metric, symbol Device:R
- removed R16: 4.7k, Resistor_SMD:R_0603_1608Metric, symbol Device:R
- added C49: 100uF, Capacitor_SMD:C_0603_1608Metric, symbol Device:C
- added TP22, TP24: USB_DN, TestPoint:TestPoint_Pad_1.0x1.0mm, symbol Connector:TestPoint
- added TP23, TP25: USB_DP, TestPoint:TestPoint_Pad_1.0x1.0mm, symbol Connector:TestPoint
- added TP26: STM32_SWCLK, TestPoint:TestPoint_Pad_1.0x1.0mm, symbol Connector:TestPoint
- added TP27: STM32_SWDIO, TestPoint:TestPoint_Pad_1.0x1.0mm, symbol Connector:TestPoint
- added TP28: STM32_TRACESWO, TestPoint:TestPoint_Pad_1.0x1.0mm, symbol Connector:TestPoint
- added TP29: STM32_NRST, TestPoint:TestPoint_Pad_1.0x1.0mm, symbol Connector:TestPoint
- added TP30, TP31: Motor1, TestPoint:TestPoint_Pad_1.0x1.0mm, symbol Connector:TestPoint
- added TP32, TP33: Servo1, TestPoint:TestPoint_Pad_1.0x1.0mm, symbol Connector:TestPoint
- added TP34, TP35: ESP32_EN, TestPoint:TestPoint_Pad_1.0x1.0mm, symbol Connector:TestPoint
- added TP36, TP37: ESP32_BOOT, TestPoint:TestPoint_Pad_1.0x1.0mm, symbol Connector:TestPoint
- added TP38, TP39: ESP32_RX, TestPoint:TestPoint_Pad_1.0x1.0mm, symbol Connector:TestPoint
- added TP40, TP43: ESP32_TX, TestPoint:TestPoint_Pad_1.0x1.0mm, symbol Connector:TestPoint
- added TP42: STM32_GND, TestPoint:TestPoint_Pad_1.0x1.0mm, symbol Connector:TestPoint
- added TP44, TP45: LED_ARRAY, TestPoint:TestPoint_Pad_1.0x1.0mm, symbol Connector:TestPoint
- added TP46, TP47: BUZZ, TestPoint:TestPoint_Pad_1.0x1.0mm, symbol Connector:TestPoint
- added TP48, TP49: VMON, TestPoint:TestPoint_Pad_1.0x1.0mm, symbol Connector:TestPoint
- added TP50: ServoPWM, TestPoint:TestPoint_Pad_1.0x1.0mm, symbol Connector:TestPoint
- added TP51, TP57, TP60, TP64, TP67: 5V, TestPoint:TestPoint_Pad_1.0x1.0mm, symbol Connector:TestPoint
- added TP52, TP53: 5V SIG, TestPoint:TestPoint_Pad_1.0x1.0mm, symbol Connector:TestPoint
- added TP54: DOUT1, TestPoint:TestPoint_Pad_1.0x1.0mm, symbol Connector:TestPoint
- added TP55: DIN1, TestPoint:TestPoint_Pad_1.0x1.0mm, symbol Connector:TestPoint
- added TP56, TP62, TP66, TP69: GND, TestPoint:TestPoint_Pad_1.0x1.0mm, symbol Connector:TestPoint
- added TP58: 5V OUTPUT, TestPoint:TestPoint_Pad_2.0x2.0mm, symbol Connector:TestPoint
- added TP59: GND OUTPUT, TestPoint:TestPoint_Pad_2.0x2.0mm, symbol Connector:TestPoint
- added TP61: DOUT2, TestPoint:TestPoint_Pad_1.0x1.0mm, symbol Connector:TestPoint
- added TP63: DOUT3, TestPoint:TestPoint_Pad_1.0x1.0mm, symbol Connector:TestPoint
- added TP65: DIN2, TestPoint:TestPoint_Pad_1.0x1.0mm, symbol Connector:TestPoint
- added TP68: DIN3, TestPoint:TestPoint_Pad_1.0x1.0mm, symbol Connector:TestPoint
- added TP70: 3.3V OUTPUT, TestPoint:TestPoint_Pad_2.0x2.0mm, symbol Connector:TestPoint
- added TP71: 3.3V INPUT, TestPoint:TestPoint_Pad_1.0x1.0mm, symbol Connector:TestPoint
- added TP72: 3.3V INPUT, TestPoint:TestPoint_Pad_2.0x2.0mm, symbol Connector:TestPoint
- added TP73: ServoVCC, TestPoint:TestPoint_Pad_1.0x1.0mm, symbol Connector:TestPoint
- added TP74: ServoGND, TestPoint:TestPoint_Pad_1.0x1.0mm, symbol Connector:TestPoint
Connections:
- net +3.3V: now also U4.2 (GND), U4.6 (VCCB), TP70.1, TP71.1, TP72.1; no longer U4.1 (VCCA), U4.5 (DIR)
- net +5V: now also U4.1 (VCCA), TP58.1; no longer C44.2, C46.2, C47.2, C48.2, LED1.3 (VDD), LED2.3 (VDD), LED3.3 (VDD), LED4.3 (VDD), U4.6 (VCCB)
- net BATT_SW+: now also C49.2, TP73.1
- net GND: now also U4.5 (DIR), C49.1, TP42.1, TP59.1, TP74.1; no longer C46.1, C47.1, C48.1, LED1.1 (GND), LED2.1 (GND), LED3.1 (GND), LED4.1 (GND), U4.2 (GND)
- net at LED4.2 (DIN): now also TP68.1; no longer LED3.4 (DOUT)
- net at R19.2: now also U4.3 (A); no longer U4.4 (B)
- net at LED1.2 (DIN): now also TP53.1; no longer R9.1
- net at LED1.4 (DOUT): now also TP54.1; no longer LED2.2 (DIN)
- net at LED3.2 (DIN): now also TP65.1; no longer LED2.4 (DOUT)
- net STM32_NRST: no longer names the net of C60.2, U2.7 (PG10-NRST)
- net STM32_NRST: now also TP29.1
- net STM32_PA0: no longer names the net of C52.2, R18.1, U6.8 (EN)
- net STM32_PA0: now also TP34.1; no longer U2.12 (PA0)
- net STM32_PA1: no longer names the net of U6.23 (IO9)
- net STM32_PA1: now also TP36.1; no longer U2.13 (PA1)
- net STM32_PA2: no longer names the net of U2.14 (PA2)
- net STM32_PA2: now also TP39.1; no longer U6.30 (RXD0)
- net STM32_PA3: no longer names the net of U6.31 (TXD0)
- net STM32_PA3: now also TP40.1; no longer U2.17 (PA3)
- net STM32_PA9 renamed STM32_USB_VBUS
- net STM32_PB0: no longer names the net of C71.2, R25.2, R26.2
- net STM32_PB0: now also TP48.1; no longer U2.24 (PB0)
- net STM32_PB11 renamed BARO_INT
- net STM32_PB12 renamed BARO_CSB
- net STM32_PB13 renamed SENSOR_SCL
- net STM32_PB14 renamed SENSOR_SDO
- net STM32_PB15 renamed SENSOR_SDA
- net STM32_PC2: no longer names the net of R12.1
- net STM32_PC2: now also TP30.1; no longer U2.10 (PC2)
- net STM32_PC3: no longer names the net of U2.11 (PC3)
- net STM32_PC3: now also TP33.1
- net STM32_PC4: no longer names the net of U2.22 (PC4)
- net STM32_PC4: now also TP45.1; no longer U4.3 (A)
- net STM32_PC5: no longer names the net of U2.23 (PC5)
- net STM32_PC5: now also TP47.1; no longer R27.1
- net STM32_PC6 renamed IMU_INT2
- net STM32_PC7 renamed IMU_INT1
- net STM32_PC8 renamed IMU_CS
- net STM32_SWCLK: no longer names the net of U2.50 (PA14)
- net STM32_SWCLK: now also TP26.1
- net STM32_SWDIO: no longer names the net of U2.49 (PA13)
- net STM32_SWDIO: now also TP27.1
- net STM32_TRACESWO: no longer names the net of U2.56 (PB3)
- net STM32_TRACESWO: now also TP28.1
- net STM32_USB_DN: no longer names the net of D6.6 (I/O1)
- net STM32_USB_DN: now also TP22.1; no longer U2.45 (PA11)
- net STM32_USB_DP: no longer names the net of U2.46 (PA12)
- net STM32_USB_DP: now also TP25.1; no longer D6.4 (I/O2)
- new net: LED4.3 (VDD), TP67.1
- new net: LED4.1 (GND), TP69.1
- new net: TP44.1, U4.4 (B)
- new net: TP32.1, TP50.1
- new net: C48.1, LED3.1 (GND), TP66.1
- new net: C48.2, LED3.3 (VDD), TP64.1
- new net: R27.1, TP46.1
- new net: TP38.1, U6.30 (RXD0)
- new net: C46.1, LED1.1 (GND), TP56.1
- new net: C46.2, LED1.3 (VDD), TP51.1
- new net: LED3.4 (DOUT), TP63.1
- new net: D6.4 (I/O2), TP23.1
- new net: R9.1, TP52.1
- new net: TP35.1, U2.12 (PA0)
- new net: C44.2, TP57.1
- new net: C47.1, LED2.1 (GND), TP62.1
- new net: C47.2, LED2.3 (VDD), TP60.1
- new net: TP31.1, U2.10 (PC2)
- new net: TP37.1, U2.13 (PA1)
- new net: TP43.1, U2.17 (PA3)
- new net: TP49.1, U2.24 (PB0)
- new net: TP24.1, U2.45 (PA11)
- new net: LED2.2 (DIN), TP55.1
- new net: LED2.4 (DOUT), TP61.1
- no-connect marks 41 -> 42
Other:
- note added: "Connect to 5v output"
- note added: "Connect to 5v sig"
- note added: "Servo 1"
- note removed: "ESP32-C3 DEBUG"
- note removed: "MOTOR 1"
- note removed: "MOTOR 2"
- note removed: "Motor 2"
- note removed: "USB"
- note removed: "VBUS"
- moved on the sheet: BUZZER2, C38, C39, C40, C41, C44, C45, C46, C47, C48, C68, D1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
