File: LSwarm Firefly/LSwarm Firefly.kicad_sch (KiCad schematic)
At the start: 134 parts, among them J3 JST / BT2.0 Connector, J4 Conn_01x02_Pin, Q1 AO3400A, Q7 AO3407A, SW1 MSK12C02, SW3 SKRPACE010, U1 LSM6DSRTR, U12 AP2112K-3.3, U2 STM32G473RCT6, U3 TPS61023DRLR, U4 SN74LVC1T45DBVR, U5 BMP581, U6 ESP32-C3-MINI-1U-N4

Commit message: sync
Parts:
- removed D1: SS14, Diode_SMD:D_SMA, symbol Diode:SS14
- removed J4: Conn_01x02_Pin, Connector_PinHeader_2.54mm:PinHeader_1x02_P2.54mm_Vertical, symbol Connector:Conn_01x02_Pin
- removed Q1: AO3400A, Package_TO_SOT_SMD:SOT-23, symbol Transistor_FET:AO3400A
- removed R11: 4.7k, Resistor_SMD:R_0603_1608Metric, symbol Device:R
- removed R12: 100, Resistor_SMD:R_0603_1608Metric, symbol Device:R
- removed TP22, TP24: USB_DN, TestPoint:TestPoint_Pad_1.0x1.0mm, symbol Connector:TestPoint
- removed TP23, TP25: USB_DP, TestPoint:TestPoint_Pad_1.0x1.0mm, symbol Connector:TestPoint
- removed TP30, TP31: Motor1, TestPoint:TestPoint_Pad_1.0x1.0mm, symbol Connector:TestPoint
- added C61, C69, C70: 100nF, Capacitor_SMD:C_0603_1608Metric, symbol Device:C
- added C72: 10uF, Capacitor_SMD:C_0603_1608Metric, symbol Device:C
- added C73: 1uF, Capacitor_SMD:C_0603_1608Metric, symbol Device:C
- added R34, R43: 10k, Resistor_SMD:R_0603_1608Metric, symbol Device:R
- added R35, R39: 47k, Resistor_SMD:R_0603_1608Metric, symbol Device:R
- added TP100, TP94: M_INHB, TestPoint:TestPoint_Pad_1.0x1.0mm, symbol Connector:TestPoint
- added TP101, TP95: M_INHA, TestPoint:TestPoint_Pad_1.0x1.0mm, symbol Connector:TestPoint
- added TP102, TP103: M_nFAULT, TestPoint:TestPoint_Pad_1.0x1.0mm, symbol Connector:TestPoint
- added TP104, TP85: M_SOB, TestPoint:TestPoint_Pad_1.0x1.0mm, symbol Connector:TestPoint
- added TP41, TP96: M_INLC, TestPoint:TestPoint_Pad_1.0x1.0mm, symbol Connector:TestPoint
- added TP75, TP76: STATUS, TestPoint:TestPoint_Pad_1.0x1.0mm, symbol Connector:TestPoint
- added TP79, TP80, TP81: GND INPUT, TestPoint:TestPoint_Pad_1.0x1.0mm, symbol Connector:TestPoint
- added TP83, TP86: M_SOA, TestPoint:TestPoint_Pad_1.0x1.0mm, symbol Connector:TestPoint
- added TP84: M_SOC, TestPoint:TestPoint_Pad_1.0x1.0mm, symbol Connector:TestPoint
- added TP87: MotorA, TestPoint:TestPoint_Pad_1.0x1.0mm, symbol Connector:TestPoint
- added TP88: MotorB, TestPoint:TestPoint_Pad_1.0x1.0mm, symbol Connector:TestPoint
- added TP89: MotorC, TestPoint:TestPoint_Pad_1.0x1.0mm, symbol Connector:TestPoint
- added TP90, TP98: M_INLA, TestPoint:TestPoint_Pad_1.0x1.0mm, symbol Connector:TestPoint
- added TP91, TP92: M_nSleep, TestPoint:TestPoint_Pad_1.0x1.0mm, symbol Connector:TestPoint
- added TP93, TP99: M_INHC, TestPoint:TestPoint_Pad_1.0x1.0mm, symbol Connector:TestPoint
- added TP97: M_INLB, TestPoint:TestPoint_Pad_1.0x1.0mm, symbol Connector:TestPoint
- added U7: DRV8311HRRWR, easyeda2kicad:QFN-24_L3.0-W3.0-P0.40-TL-EP1.9_TI_RRW0024A, symbol easyeda2kicad:DRV8311HRRWR
- TP42: value STM32_GND -> M_INLB
- TP57: value 5V -> M_SOC
- TP58, TP59, TP70, TP72: footprint TestPoint:TestPoint_Pad_2.0x2.0mm -> TestPoint:TestPoint_Pad_1.0x1.0mm
Connections:
- net +3.3V: now also R43.2
- net +5V: now also C44.2
- net BATT_SW+: now also C69.2, C70.1, U7.7 (VIN_AVDD), U7.8 (VM)
- net GND: now also C61.2, C72.2, C73.1, R34.1, R35.1, R39.1, TP79.1, TP80.1, TP81.1, U7.16 (AGND), U7.21 (GAIN), U7.25 (EP), U7.9 (PGND); no longer TP42.1
- net IMU_CS: now also U2.43 (PA9); no longer U2.40 (PC8)
- net IMU_INT1: now also U2.42 (PA8); no longer U2.39 (PC7)
- net IMU_INT2: now also U2.41 (PC9); no longer U2.38 (PC6)
- net STM32_USB_VBUS: now also U2.44 (PA10); no longer U2.43 (PA9)
- net USB_DP: now reaches U2.46 (PA12)
- net USB_DP: now also D6.4 (I/O2)
- net USB_DN: now reaches D6.6 (I/O1)
- net USB_DN: now also U2.45 (PA11)
- net at TP57.1: now also U2.25 (PB1); no longer C44.2
- net at U2.11 (PC3): no longer TP33.1
- net at U2.18 (PA4): now also TP91.1
- net at U2.20 (PA6): now also TP83.1
- net at U2.21 (PA7): now also TP104.1
- net at U2.52 (PC10): now also TP90.1
- net at U2.53 (PC11): now also TP42.1
- net at U2.54 (PC12): now also TP41.1
- net at U2.57 (PB4): now also TP33.1
- net at U2.59 (PB6): now also TP102.1
- net STM32_PB7: no longer names the net of R10.2
- net STM32_PB7: now also TP76.1; no longer U2.60 (PB7)
- new net: TP86.1, U7.5 (SOA)
- new net: C73.2, R43.1, TP103.1, U7.1 (nFAULT), U7.17 (AVDD)
- new net: TP87.1, U7.10 (OUTA)
- new net: TP88.1, U7.11 (OUTB)
- new net: TP89.1, U7.12 (OUTC)
- new net: TP99.1, U7.13 (INHC)
- new net: TP100.1, U7.14 (INHB)
- new net: TP101.1, U7.15 (INHA)
- new net: TP98.1, U7.18 (INLA)
- new net: TP97.1, U7.19 (INLB)
- new net: C61.1, U7.2 (CSAREF)
- new net: TP96.1, U7.20 (INLC)
- new net: R39.2, U7.22 (SLEW)
- new net: R35.2, U7.23 (MODE)
- new net: R34.2, TP92.1, U7.24 (nSLEEP)
- new net: TP84.1, U7.3 (SOC)
- new net: TP85.1, U7.4 (SOB)
- new net: C69.1, U7.6 (CP)
- new net: TP93.1, U2.40 (PC8)
- new net: C70.2, C72.1
- new net: TP75.1, U2.60 (PB7)
- new net: TP95.1, U2.38 (PC6)
- new net: TP94.1, U2.39 (PC7)
Other:
- note removed: "+"
- note removed: "STATUS"
- moved on the sheet: BUZZER2, C49, R27, R42, TP32, TP33, TP46, TP50, TP71, TP73, TP74

Commit message: sync
Parts:
- removed C27: 10nF, Capacitor_SMD:C_0603_1608Metric, symbol Device:C
- removed D6: USBLC6-2SC6_C2687116, easyeda2kicad:SOT-23-6_L2.9-W1.6-P0.95-LS2.8-BL, symbol easyeda2kicad:USBLC6-2SC6_C2687116
- removed J3: JST / BT2.0 Connector, Connector_JST:JST_PH_S2B-PH-K_1x02_P2.00mm_Horizontal, symbol Connector:Conn_01x02_Socket
- removed R14, R15: 100k, Resistor_SMD:R_0603_1608Metric, symbol Device:R
- removed R38, R41: 5.1k, Resistor_SMD:R_0603_1608Metric, symbol Device:R
- removed TP100, TP94: M_INHB, TestPoint:TestPoint_Pad_1.0x1.0mm, symbol Connector:TestPoint
- removed TP101, TP95: M_INHA, TestPoint:TestPoint_Pad_1.0x1.0mm, symbol Connector:TestPoint
- removed TP102, TP103: M_nFAULT, TestPoint:TestPoint_Pad_1.0x1.0mm, symbol Connector:TestPoint
- removed TP104, TP85: M_SOB, TestPoint:TestPoint_Pad_1.0x1.0mm, symbol Connector:TestPoint
- removed TP32, TP33: Servo1, TestPoint:TestPoint_Pad_1.0x1.0mm, symbol Connector:TestPoint
- removed TP41, TP96: M_INLC, TestPoint:TestPoint_Pad_1.0x1.0mm, symbol Connector:TestPoint
- removed TP42, TP97: M_INLB, TestPoint:TestPoint_Pad_1.0x1.0mm, symbol Connector:TestPoint
- removed TP48, TP49: VMON, TestPoint:TestPoint_Pad_1.0x1.0mm, symbol Connector:TestPoint
- removed TP57, TP84: M_SOC, TestPoint:TestPoint_Pad_1.0x1.0mm, symbol Connector:TestPoint
- removed TP70: 3.3V OUTPUT, TestPoint:TestPoint_Pad_1.0x1.0mm, symbol Connector:TestPoint
- removed TP81: GND INPUT, TestPoint:TestPoint_Pad_1.0x1.0mm, symbol Connector:TestPoint
- removed TP83, TP86: M_SOA, TestPoint:TestPoint_Pad_1.0x1.0mm, symbol Connector:TestPoint
- removed TP90, TP98: M_INLA, TestPoint:TestPoint_Pad_1.0x1.0mm, symbol Connector:TestPoint
- removed TP91, TP92: M_nSleep, TestPoint:TestPoint_Pad_1.0x1.0mm, symbol Connector:TestPoint
- removed TP93, TP99: M_INHC, TestPoint:TestPoint_Pad_1.0x1.0mm, symbol Connector:TestPoint
- removed USB2: USB-TYPE-C-018, easyeda2kicad:USB-C_SMD-TYPE-C-31-M-12, symbol easyeda2kicad:USB-TYPE-C-018
- added J1, J2: Conn_01x02_Socket, Connector_PinHeader_1.00mm:PinHeader_1x02_P1.00mm_Vertical, symbol Connector:Conn_01x02_Socket
- added U8: DW3110TR13, easyeda2kicad:WLCSP-53_L3.5-W3.0_DW3110TR13, symbol easyeda2kicad:DW3110TR13
Connections:
- net BATT+: now also J1.1 (Pin_1)
- net GND: now also J2.2 (Pin_2)
- net M_SOA: now reaches U7.5 (SOA)
- net M_SOA: now also U2.20 (PA6)
- net M_INLA: now reaches U2.52 (PC10)
- net M_INLA: now also U7.18 (INLA)
- net M_nSLEEP: now reaches U2.18 (PA4)
- net M_nSLEEP: now also R34.2, U7.24 (nSLEEP)
- net V_MON: now reaches C71.2, R25.2, R26.2
- net V_MON: now also U2.24 (PB0)
- net M_nFAULT: now reaches C73.2, R43.1, U7.1 (nFAULT), U7.17 (AVDD)
- net M_nFAULT: now also U2.59 (PB6)
- net M_INHC: now reaches U7.13 (INHC)
- net M_INHC: now also U2.40 (PC8)
- net M_INHB: now reaches U7.14 (INHB)
- net M_INHB: now also U2.39 (PC7)
- net M_INHA: now reaches U7.15 (INHA)
- net M_INHA: now also U2.38 (PC6)
- net M_INLB: now reaches U7.19 (INLB)
- net M_INLB: now also U2.53 (PC11)
- net M_INLC: now reaches U7.20 (INLC)
- net M_INLC: now also U2.54 (PC12)
- net M_SOC: now reaches U7.3 (SOC)
- net M_SOC: now also U2.25 (PB1)
- net M_SOB: now reaches U7.4 (SOB)
- net M_SOB: now also U2.21 (PA7)
- net SERVO_PWM: now reaches TP50.1
- net SERVO_PWM: now also U2.57 (PB4)
- net USB_DN: no longer names the net of U2.45 (PA11)
- net USB_DP: no longer names the net of U2.46 (PA12)
- new net: J1.2 (Pin_2), J2.1 (Pin_1)
- no-connect marks 42 -> 40
Other:
- note added: "1s lipos"
- note added: "Brushless Motor"
- note added: "Servo"
- note removed: "ESD Protection"
- note removed: "Motor 1"
- note removed: "Servo 1"
- note removed: "USB-C Connector"
- note removed: "VBUS Divider"
- moved on the sheet: BUZZER2, C1, C38, C39, C40, C41, C42, C43, C44, C45, C46, C47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

Commit message: sync
Parts:
- added C2: 0603CG2R0C500NT, easyeda2kicad:C0603, symbol easyeda2kicad:0603CG2R0C500NT
- added C74, C75, C79, C80, C81: 100nf, Capacitor_SMD:C_0603_1608Metric, symbol Device:C
- added C76: 10uF, Capacitor_SMD:C_0603_1608Metric, symbol Device:C
- added C77, C78: 3.3pF, Capacitor_SMD:C_0603_1608Metric, symbol Device:C
- added JP1: U.FL-R-SMT-1, easyeda2kicad:RF-SMD_FRF05002-JSS103M, symbol easyeda2kicad:U.FL-R-SMT-1
- added L1: MPZ2012S601AT000, easyeda2kicad:L0805, symbol easyeda2kicad:MPZ2012S601AT000
- added R1: RC0402FR-0749R9L, easyeda2kicad:R0402, symbol easyeda2kicad:RC0402FR-0749R9L
- added R38, R41: 10k, Resistor_SMD:R_0603_1608Metric, symbol Device:R
- added R40, R44: 100k, Resistor_SMD:R_0603_1608Metric, symbol Device:R
- added TP81: SYNC, TestPoint:TestPoint_Pad_1.0x1.0mm, symbol Connector:TestPoint
- added U10: BLM03PG330SN1D, easyeda2kicad:L0201, symbol easyeda2kicad:BLM03PG330SN1D
- added U11: BU03, easyeda2kicad:WIRELM-SMD_BU03, symbol easyeda2kicad:BU03
- added U9: 8Y38472012, easyeda2kicad:CRYSTAL-SMD_4P-L2.0-W1.6-BL, symbol easyeda2kicad:8Y38472012
Connections:
- net +3.3V: now also U8.B13 (VDD1), U8.B15 (VDD2b), U8.D15 (VDD3), L1.2, R38.1, R41.1, U10.2
- net GND: now also U8.A14 (VSS1), U8.A2 (VSS), U8.B11 (VSS1), U8.B3 (VSS), U8.C10 (VSS1), U8.C12 (VSS3), U8.C6 (VSS), U8.C8 (VSS1), U8.D11 (VSS2), U8.D13 (VSS3), U8.D5 (VSS), U8.D7 (VSS), U8.D9 (VSS1), U8.E10 (GND), U8.E12 (GND), U8.E14 (VSS2), U8.E6 (GND), U8.F7 (GND), U8.F9 (GND), U8.G10 (GND), U8.G6 (GND), U8.H1 (GND), U8.H13 (GND), U8.H3 (GND), U8.H7 (GND), U8.H9 (GND), C74.1, C75.1, C76.2, C77.2, C78.2, C79.2, C80.2, C81.2, JP1.2 (GND), JP1.3 (GND), R1.1, R40.2, R44.1, U11.16 (GND), U11.24 (GND), U11.8 (GND), U9.2 (GND), U9.4 (GND)
- net DW_RST: now reaches U8.A10 (RSTn)
- net DW_RST: now also U6.16 (IO10), R38.2, U11.3 (RSTN)
- net at U8.A4 (VIO_D): now also C75.2
- net DW_MISO: now reaches U8.A6 (SPICDO(SPIMISO))
- net DW_MISO: now also U6.18 (IO4), U11.19 (MISO)
- net DW_CLK: now reaches U8.A8 (SPICK)
- net DW_CLK: now also U6.20 (IO6), U11.20 (CLK)
- net DW_IRQ: now reaches U8.B1 (IRQ)
- net DW_IRQ: now also U6.6 (IO3), R40.1, R44.2, U11.22 (IRQ)
- net DW_Sn: now reaches U8.B5 (SPICSn)
- net DW_Sn: now also U6.21 (IO7), R41.2, U11.17 (CSN)
- net DW_MOSI: now reaches U8.B7 (SPIDCI(SPIMOSI))
- net DW_MOSI: now also U6.19 (IO5), U11.18 (MOSI)
- net DW_WAKEUP: now reaches U8.B9 (WAKEUP)
- net DW_WAKEUP: now also U6.13 (IO1), U11.2 (WAKEUP)
- net at U8.C14 (VTX_D): now also C74.2
- net at U8.F15 (VDD2a): now also U10.1
- net at U8.G14 (XTO): now also C78.1, U9.3 (OSC2)
- net at U8.G2 (GPIO07/SYNC): now also TP81.1
- net at U8.H11 (RF1): now also C2.2
- net at U8.H15 (XTI): now also C77.1, U9.1 (OSC1)
- net at U8.H5 (RF2): now also R1.2
- new net: C2.1, JP1.1 (SIG)
- new net UW_3.3V: C76.1, C79.1, C80.1, C81.1, L1.1, U11.5 (VDD), U11.6 (VCC), U11.7 (VCC)
- no-connect marks 40 -> 52
Other:
- note added: "UWB ANCHOR"
- note added: "UWB TAG"
- moved on the sheet: BUZZER2, C38, C39, C40, C41, C52, C61, C62, C63, C64, C68, C69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

Commit message: sync
Parts:
- removed C2: 0603CG2R0C500NT, easyeda2kicad:C0603, symbol easyeda2kicad:0603CG2R0C500NT
- removed C74, C75: 100nf, Capacitor_SMD:C_0603_1608Metric, symbol Device:C
- removed C77, C78: 3.3pF, Capacitor_SMD:C_0603_1608Metric, symbol Device:C
- removed JP1: U.FL-R-SMT-1, easyeda2kicad:RF-SMD_FRF05002-JSS103M, symbol easyeda2kicad:U.FL-R-SMT-1
- removed R1: RC0402FR-0749R9L, easyeda2kicad:R0402, symbol easyeda2kicad:RC0402FR-0749R9L
- removed R38: 10k, Resistor_SMD:R_0603_1608Metric, symbol Device:R
- removed R40: 100k, Resistor_SMD:R_0603_1608Metric, symbol Device:R
- removed TP81: SYNC, TestPoint:TestPoint_Pad_1.0x1.0mm, symbol Connector:TestPoint
- removed U10: BLM03PG330SN1D, easyeda2kicad:L0201, symbol easyeda2kicad:BLM03PG330SN1D
- removed U8: DW3110TR13, easyeda2kicad:WLCSP-53_L3.5-W3.0_DW3110TR13, symbol easyeda2kicad:DW3110TR13
- removed U9: 8Y38472012, easyeda2kicad:CRYSTAL-SMD_4P-L2.0-W1.6-BL, symbol easyeda2kicad:8Y38472012
Connections:
- no-connect marks 52 -> 44
Other:
- note removed: "UWB TAG"
- moved on the sheet: C38, C39, C40, C41, C68, L1, R29, R30, R31, R41, R44, U1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

Commit message: sync
Parts:
- removed SW1: MSK12C02, easyeda2kicad:SW-TH_MSK12C02, symbol easyeda2kicad:MSK12C02
- removed TP75: STATUS, TestPoint:TestPoint_Pad_1.0x1.0mm, symbol Connector:TestPoint
- added C77, C82: 100nF, Capacitor_SMD:C_0603_1608Metric, symbol Device:C
- added C78, C83: 1uF, Capacitor_SMD:C_0603_1608Metric, symbol Device:C
- added R38, R40, R45, R46: 4.7k, Resistor_SMD:R_0603_1608Metric, symbol Device:R
- added SW2: MINI MSK12CO2, easyeda2kicad:SW-SMD_MSK12CO2, symbol easyeda2kicad:MINIMSK12CO2
- added TP77: STATUS, TestPoint:TestPoint_Pad_1.0x1.0mm, symbol Connector:TestPoint
- added U8, U9: MMC5603NJ, easyeda2kicad:FLIPCHIP-4_L0.8-W0.8-R2-C2-P0.40-TL, symbol easyeda2kicad:MMC5603NJ
Connections:
- net +3.3V: now also C77.1, C82.1, R38.2, R40.2, R45.2, R46.2, U8.B1 (VDD), U9.B1 (VDD)
- net BATT+: now also C69.2, C70.1, U7.7 (VIN_AVDD), U7.8 (VM)
- net BATT_SW+: no longer C69.2, C70.1, U7.7 (VIN_AVDD), U7.8 (VM)
- net GND: now also C78.2, C83.2, SW2.3, U8.A1 (VSA), U9.A1 (VSA)
- net ESP32_MAG_SDA: now reaches U6.26 (IO18)
- net ESP32_MAG_SDA: now also R45.1, U9.B2 (SDA)
- net ESP32_MAG_SCL: now reaches U6.27 (IO19)
- net ESP32_MAG_SCL: now also R46.1, U9.A2 (SCL)
- net STM_MAG_SDA: now reaches U2.60 (PB7)
- net STM_MAG_SDA: now also R38.1, U8.B2 (SDA)
- net STM_MAG_SCL: now reaches U2.51 (PA15)
- net STM_MAG_SCL: now also R40.1, U8.A2 (SCL)
- net at U2.58 (PB5): now also TP77.1
- net at R17.1: now also SW2.2
- new net: C82.2, C83.1
- new net: C77.2, C78.1
- no-connect marks 44 -> 43
Other:
- note added: "ESP32 MAG"
- note added: "STM MAG"
- moved on the sheet: Q7
